File: KiCad/Hexapod_bot.kicad_sch (KiCad schematic)
At the start: 3 parts, among them J1 Ras Pi 4 Interface

Commit message: Finished Rev 1 of the PCB
Parts:
- added D1: LED Blue, LED_SMD:LED_0603_1608Metric_Pad1.05x0.95mm_HandSolder, symbol Device:LED
- added H1, H2, H3, H4: MountingHole_Pad, Spiderbot:MountingHole_2.5mm_Pad_TopBottom, symbol Mechanical:MountingHole_Pad
- added J2: Leg Switches, Connector_PinSocket_2.54mm:PinSocket_2x06_P2.54mm_Vertical, symbol Connector_Generic:Conn_02x06_Odd_Even
- added R3: 1.2k, Resistor_SMD:R_0603_1608Metric_Pad0.98x0.95mm_HandSolder, symbol Device:R_US
- added R4, R5, R6, R7, R8, R9: 10k, Resistor_SMD:R_0603_1608Metric_Pad0.98x0.95mm_HandSolder, symbol Device:R_US
- J1: footprint (none) -> Connector_PinSocket_2.54mm:PinSocket_2x20_P2.54mm_Vertical; Link (none) -> https://www.digikey.com/en/products/detail/sparkfun-electro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
- R1: renamed from R7; footprint (none) -> Resistor_SMD:R_0603_1608Metric_Pad0.98x0.95mm_HandSolder
- R2: renamed from R6; footprint (none) -> Resistor_SMD:R_0603_1608Metric_Pad0.98x0.95mm_HandSolder
Connections:
- net 3V3_pi: now also J2.1 (Pin_1), J2.11 (Pin_11), J2.3 (Pin_3), J2.5 (Pin_5), J2.7 (Pin_7), J2.9 (Pin_9)
- net GND: now also J1.39 (Pin_39), D1.1 (K), H1.1, H2.1, H3.1, H4.1, R4.2, R5.2, R6.2, R7.2, R8.2, R9.2
- net BattLow: now reaches J1.13 (Pin_13)
- net at J1.27 (Pin_27): now also J2.2 (Pin_2), R6.1
- net at J1.29 (Pin_29): now also J2.4 (Pin_4), R9.1
- net at J1.31 (Pin_31): now also J2.6 (Pin_6), R5.1
- net at J1.33 (Pin_33): now also J2.8 (Pin_8), R8.1
- net at J1.35 (Pin_35): now also J2.10 (Pin_10), R4.1
- net at J1.37 (Pin_37): now also J2.12 (Pin_12), R7.1
- net at J1.8 (Pin_8): now also R3.2
- net CLK renamed CLK_3V3
- new net: D1.2 (A), R3.1
- no-connect marks 0 -> 25
Other:
- moved on the sheet: J1, R1, R2
