File: KiCad/imu.kicad_sch (KiCad schematic)
At the start: 5 parts, among them U2 LSM6DSO32TR

Commit message: Finished Rev 1 of the PCB
Parts:
- C15: renamed from C3; value 100nF -> 0.1uF; footprint (none) -> Capacitor_SMD:C_0603_1608Metric_Pad1.08x0.95mm_HandSolder
- C16: value 100nF -> 0.1uF; footprint (none) -> Capacitor_SMD:C_0603_1608Metric_Pad1.08x0.95mm_HandSolder
- R49: renamed from R18; footprint (none) -> Resistor_SMD:R_0603_1608Metric_Pad0.98x0.95mm_HandSolder
- R50: renamed from R17; footprint (none) -> Resistor_SMD:R_0603_1608Metric_Pad0.98x0.95mm_HandSolder
- U8: renamed from U2; footprint LGA-14L_2P5X3X0P83_STM -> Spiderbot:LGA-14L_2P5X3X0P83_STM; Link (none) -> https://www.digikey.com/en/products/detail/stmicroelectroni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
Connections:
- no-connect marks 6 -> 4
Other:
- moved on the sheet: C16
