File: KiCad/servo_control.kicad_sch (KiCad schematic)
At the start: 47 parts, among them J10 Conn_01x03, J11 Conn_01x03, J12 Conn_01x03, J13 Conn_01x03, J14 Conn_01x03, J15 Conn_01x03, J16 Conn_01x03, J17 Conn_01x03, J18 Conn_01x03, J19 Conn_01x03, J2 Conn_01x03, J20 Conn_01x03, J21 Conn_01x03, J22 Conn_01x03, J23 Conn_01x03, J3 Conn_01x03, J4 Conn_01x03, J5 Conn_01x03, J6 Conn_01x03, J7 Conn_01x03, J8 Conn_01x03, J9 Conn_01x03, Q2 BSS138, U1 PCA9685PW, U5 LSF0102DCUR, U7 PCA9685PW

Commit message: Finished Rev 1 of the PCB
Parts:
- removed C14: 0.1mF, symbol Device:C
- removed R12, R13: R_US, symbol Device:R_US
- removed RN1, RN2: 10k, Resistor_THT:R_Array_SIP7, symbol Device:R_Network06_US
- removed U5: LSF0102DCUR, DCU0008A_N, symbol Alecs_Lib:LSF0102DCUR
- added Q3, Q4: BSS138, Spiderbot:SOT-23_3L_ONS, symbol Simulation_SPICE:NMOS
- added R29, R30, R31, R32, R33, R34, R35, R36, R37, R38, R39, R40, R41, R42, R43, R44, R45, R46: 10k, Resistor_SMD:R_0603_1608Metric_Pad0.98x0.95mm_HandSolder, symbol Device:R_US
- C13: renamed from C4; footprint (none) -> Capacitor_SMD:C_0603_1608Metric_Pad1.08x0.95mm_HandSolder
- C14: renamed from C17; footprint (none) -> Capacitor_SMD:C_0603_1608Metric_Pad1.08x0.95mm_HandSolder
- J10: renamed from J8; footprint (none) -> Connector_PinSocket_2.54mm:PinSocket_1x03_P2.54mm_Vertical
- J11: renamed from J9; footprint (none) -> Connector_PinSocket_2.54mm:PinSocket_1x03_P2.54mm_Vertical
- J12: renamed from J10; footprint (none) -> Connector_PinSocket_2.54mm:PinSocket_1x03_P2.54mm_Vertical
- J13: renamed from J11; footprint (none) -> Connector_PinSocket_2.54mm:PinSocket_1x03_P2.54mm_Vertical
- J14: renamed from J12; footprint (none) -> Connector_PinSocket_2.54mm:PinSocket_1x03_P2.54mm_Vertical
- J15: renamed from J13; footprint (none) -> Connector_PinSocket_2.54mm:PinSocket_1x03_P2.54mm_Vertical
- J16: renamed from J14; footprint (none) -> Connector_PinSocket_2.54mm:PinSocket_1x03_P2.54mm_Vertical
- J17: renamed from J15; footprint (none) -> Connector_PinSocket_2.54mm:PinSocket_1x03_P2.54mm_Vertical
- J18: renamed from J16; footprint (none) -> Connector_PinSocket_2.54mm:PinSocket_1x03_P2.54mm_Vertical
- J19: renamed from J17; footprint (none) -> Connector_PinSocket_2.54mm:PinSocket_1x03_P2.54mm_Vertical
- J20: renamed from J18; footprint (none) -> Connector_PinSocket_2.54mm:PinSocket_1x03_P2.54mm_Vertical
- J21: renamed from J19; footprint (none) -> Connector_PinSocket_2.54mm:PinSocket_1x03_P2.54mm_Vertical
- J22: renamed from J20; footprint (none) -> Connector_PinSocket_2.54mm:PinSocket_1x03_P2.54mm_Vertical
- J23: renamed from J21; footprint (none) -> Connector_PinSocket_2.54mm:PinSocket_1x03_P2.54mm_Vertical
- J24: renamed from J22; footprint (none) -> Connector_PinSocket_2.54mm:PinSocket_1x03_P2.54mm_Vertical
- J25: renamed from J23; footprint (none) -> Connector_PinSocket_2.54mm:PinSocket_1x03_P2.54mm_Vertical
- J4: renamed from J2; footprint (none) -> Connector_PinSocket_2.54mm:PinSocket_1x03_P2.54mm_Vertical
- J5: renamed from J3; footprint (none) -> Connector_PinSocket_2.54mm:PinSocket_1x03_P2.54mm_Vertical
- J6: renamed from J4; footprint (none) -> Connector_PinSocket_2.54mm:PinSocket_1x03_P2.54mm_Vertical
- J7: renamed from J5; footprint (none) -> Connector_PinSocket_2.54mm:PinSocket_1x03_P2.54mm_Vertical
- J8: renamed from J6; footprint (none) -> Connector_PinSocket_2.54mm:PinSocket_1x03_P2.54mm_Vertical
- J9: renamed from J7; footprint (none) -> Connector_PinSocket_2.54mm:PinSocket_1x03_P2.54mm_Vertical
- JP1, JP10, JP11, JP12, JP2, JP3, JP4, JP5, JP6, JP7, JP8, JP9: footprint (none) -> Resistor_SMD:R_0603_1608Metric_Pad0.98x0.95mm_HandSolder
- Q2: footprint (none) -> Spiderbot:SOT-23_3L_ONS; Link (none) -> https://www.digikey.com/en/products/detail/onsemi/BSS138/24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
- R47: renamed from R8; footprint (none) -> Resistor_SMD:R_0603_1608Metric_Pad0.98x0.95mm_HandSolder
- R48: renamed from R19; footprint (none) -> Resistor_SMD:R_0603_1608Metric_Pad0.98x0.95mm_HandSolder
- U6: renamed from U1; footprint SOT361-1_NXP -> Spiderbot:SOT361-1_NXP; Link (none) -> https://www.digikey.com/en/products/detail/nxp-usa-inc/PCA9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
- U7: footprint SOT361-1_NXP -> Spiderbot:SOT361-1_NXP; Link (none) -> https://www.digikey.com/en/products/detail/nxp-usa-inc/PCA9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
Connections:
- net 5V is gone; now on net 5V_pi: JP1.1 (A), JP10.1 (A), JP11.1 (A), JP12.1 (A), JP2.1 (A), JP3.1 (A), JP4.1 (A), JP5.1 (A), JP6.1 (A), JP7.1 (A), JP8.1 (A), JP9.1 (A)
- net CLK is gone; now on net SDA_5V: Q2.1 (D)
- net 3V3_pi: now also Q3.2 (G), Q4.2 (G), R41.1, R42.1, R43.1
- net 5V_pi: now also R44.1, R45.1, R46.1
- net CLK_5V: now also Q4.1 (D), R46.2; no longer Q2.3 (S)
- net GND: now also R29.2, R30.2, R31.2, R32.2, R33.2, R34.2, R35.2, R36.2, R37.2, R38.2, R39.2, R40.2
- net SCL_5V: now also Q3.1 (D), R45.2
- net SDA_5V: now also R44.2
- net servo0: now also J12.1 (Pin_1); no longer J4.1 (Pin_1)
- net servo1: now also J11.1 (Pin_1); no longer J5.1 (Pin_1)
- net servo2: now also J10.1 (Pin_1); no longer J6.1 (Pin_1)
- net servo3: now also J9.1 (Pin_1); no longer J7.1 (Pin_1)
- net servo5: now also J7.1 (Pin_1); no longer J9.1 (Pin_1)
- net servo6: now also J6.1 (Pin_1); no longer J10.1 (Pin_1)
- net servo7: now also J5.1 (Pin_1); no longer J11.1 (Pin_1)
- net servo8: now also J4.1 (Pin_1); no longer J12.1 (Pin_1)
- net at JP5.2 (B), U6.5 (A4): now also R29.1
- net at JP11.2 (B), U7.5 (A4): now also R35.1
- net at JP1.2 (B), U6.1 (A0): now also R31.1
- net at JP2.2 (B), U6.2 (A1): now also R34.1
- net at JP3.2 (B), U6.3 (A2): now also R30.1
- net at JP4.2 (B), U6.4 (A3): now also R33.1
- net at JP10.2 (B), U7.4 (A3): now also R39.1
- net at JP9.2 (B), U7.3 (A2): now also R36.1
- net at JP8.2 (B), U7.2 (A1): now also R40.1
- net at JP7.2 (B), U7.1 (A0): now also R37.1
- net A5 renamed A5_1
- net A5_1: now also R32.1; no longer JP12.2 (B), U7.24 (A5)
- new net A5_2: JP12.2 (B), R38.1, U7.24 (A5)
- new net CLK_3V3: Q4.3 (S), R43.2
- new net SCL_3V3: Q3.3 (S), R42.2
- new net SDA_3V3: Q2.3 (S), R41.2
- no-connect marks 0 -> 10
Other:
- note added: "Logic Shifters"
- note removed: "Clock Shift Check to see if it needs a pullup"
- note removed: "I2C Logic Shifter"
