File: KiCad/spower_monitor.kicad_sch (KiCad schematic)
At the start: 0 parts

Commit message: Finished Rev 1 of the PCB
Parts:
- added C11, C12: 0.1F, Capacitor_SMD:C_0603_1608Metric_Pad1.08x0.95mm_HandSolder, symbol Device:C
- added D4: LED Red, LED_SMD:LED_0603_1608Metric_Pad1.05x0.95mm_HandSolder, symbol Device:LED
- added J3: Terminal Block, Spiderbot:Terminal, symbol Alecs_Lib:Terminal
- added R17: 51k, Resistor_SMD:R_0603_1608Metric_Pad0.98x0.95mm_HandSolder, symbol Device:R_US
- added R18: 1.6k, Resistor_SMD:R_0603_1608Metric_Pad0.98x0.95mm_HandSolder, symbol Device:R_US
- added R19, R20, R22, R27: 10k, Resistor_SMD:R_0603_1608Metric_Pad0.98x0.95mm_HandSolder, symbol Device:R_US
- added R21: 750k, Resistor_SMD:R_0603_1608Metric_Pad0.98x0.95mm_HandSolder, symbol Device:R_US
- added R23: 82k, Resistor_SMD:R_0603_1608Metric_Pad0.98x0.95mm_HandSolder, symbol Device:R_US
- added R24: 1k, Resistor_SMD:R_0603_1608Metric_Pad0.98x0.95mm_HandSolder, symbol Device:R_US
- added R25: 27k, Resistor_SMD:R_0603_1608Metric_Pad0.98x0.95mm_HandSolder, symbol Device:R_US
- added R26: 30k, Resistor_SMD:R_0603_1608Metric_Pad0.98x0.95mm_HandSolder, symbol Device:R_US
- added R28: 2k, Resistor_SMD:R_0603_1608Metric_Pad0.98x0.95mm_HandSolder, symbol Device:R_US
- added U4: LM78L05_SO8, Package_SO:SOIC-8_3.9x4.9mm_P1.27mm, symbol Regulator_Linear:LM78L05_SO8
- added U5: LM393, Package_SO:SOIC-8-1EP_3.9x4.9mm_P1.27mm_EP2.29x3mm, symbol Comparator:LM393
Connections:
- new net: R20.2, R27.1, U5.5 (+)
- new net: R18.1, R19.2, R21.2, U5.1, U5.6 (-)
- new net: R22.2, R24.1, U5.7
- new net: R23.2, R25.1, U5.2 (-)
- new net: C12.1, R17.1, R19.1, R20.1, R22.1, U4.1 (OUT), U5.8 (V+)
- new net: D4.2 (A), R18.2
- new net: R17.2, R21.1, R26.1, U5.3 (+)
- new net 7.4V_batt: C11.1, J3.2, R23.1, U4.8 (IN)
- new net BattLow: R24.2, R28.2
- new net GND: C11.2, C12.2, D4.1 (K), J3.1, R25.2, R26.2, R27.2, R28.1, U4.2 (GND), U4.3 (GND), U4.6 (GND), U4.7 (GND), U5.4 (V-)
Other:
- note added: "Turns on when batt low"
