Commit message: Saying Fuck it We Ball and made a new python package!

File: ros2_ws/src/hexapod_description/urdf/hexapod.xacro (robot description, xacro)
@@ -21,12 +21,12 @@
   <xacro:macro name="leg" params="name x y angle side">
     <!-- Coxa joint -->
-    <joint name="${name}_coxa_joint" type="revolute">
+    <joint name="coxa_joint_${name}" type="revolute">
       <parent link="base_link" />
-      <child link="${name}_coxa" />
+      <child link="coxa_${name}" />
       <origin xyz="${x} ${y} 0" rpy="0 0 ${angle}" />
-      <axis xyz="0 0 1" /> <!-- Coxa rotates about the Z-axis -->
+      <axis xyz="0 0 ${side}" /> <!-- Coxa rotates about the Z-axis -->
       <limit lower="${joint_lower_limit}" upper="${joint_upper_limit}" effort="${joint_effort}" velocity="${joint_velocity}" />
     </joint>
-    <link name="${name}_coxa">
+    <link name="coxa_${name}">
       <visual>
         <geometry>
@@ -39,12 +39,12 @@
     </link>
     <!-- Femur joint -->
-    <joint name="${name}_femur_joint" type="revolute">
-      <parent link="${name}_coxa" />
-      <child link="${name}_femur" />
+    <joint name="femur_joint_${name}" type="revolute">
+      <parent link="coxa_${name}" />
+      <child link="femur_${name}" />
       <origin xyz="0.044 0 0" rpy="0 0 0" />
-      <axis xyz="0 1 0" /> <!-- Femur rotates about the Y-axis -->
+      <axis xyz="0 ${side} 0" /> <!-- Femur rotates about the Y-axis -->
       <limit lower="${joint_lower_limit}" upper="${joint_upper_limit}" effort="${joint_effort}" velocity="${joint_velocity}" />
     </joint>
-    <link name="${name}_femur">
+    <link name="femur_${name}">
       <visual>
         <geometry>
@@ -57,12 +57,12 @@
     </link>
     <!-- Tibia joint -->
-    <joint name="${name}_tibia_joint" type="revolute">
-      <parent link="${name}_femur" />
-      <child link="${name}_tibia" />
+    <joint name="tibia_joint_${name}" type="revolute">
+      <parent link="femur_${name}" />
+      <child link="tibia_${name}" />
       <origin xyz="0.08 0 0" rpy="0 0 0" />
-      <axis xyz="0 1 0" /> <!-- Tibia rotates about the Y-axis -->
+      <axis xyz="0 ${side} 0" /> <!-- Tibia rotates about the Y-axis -->
       <limit lower="${joint_lower_limit}" upper="${joint_upper_limit}" effort="${joint_effort}" velocity="${joint_velocity}" />
     </joint>
-    <link name="${name}_tibia">
+    <link name="tibia_${name}">
       <visual>
         <geometry>
@@ -75,10 +75,10 @@
     </link>
     <!-- Foot -->
-    <joint name="${name}_foot_joint" type="fixed">
-      <parent link="${name}_tibia" />
-      <child link="${name}_foot" />
-      <origin xyz="-0.08 0 -0.155" rpy="0 0 0" />
+    <joint name="foot_joint_${name}" type="fixed">
+      <parent link="tibia_${name}" />
+      <child link="foot_${name}" />
+      <origin xyz="0 0 -0.155" rpy="0 0 0" />
     </joint>
-    <link name="${name}_foot">
+    <link name="foot_${name}">
       <visual>
         <geometry>
@@ -92,9 +92,9 @@
   </xacro:macro>
   <!-- Legs -->
-  <xacro:leg name="leg0" x="-0.09" y="-0.065" angle="-2.35619" side="1" /> <!-- Back Left -->
-  <xacro:leg name="leg1" x="0.0" y="-0.09" angle="-1.5708" side="1" />     <!-- Left -->
-  <xacro:leg name="leg2" x="0.09" y="-0.065" angle="-0.7854" side="1" />   <!-- Front Left -->
-  <xacro:leg name="leg3" x="-0.09" y="0.065" angle="2.35619" side="-1" />  <!-- Back Right -->
-  <xacro:leg name="leg4" x="0.0" y="0.09" angle="1.5708" side="-1" />      <!-- Right -->
-  <xacro:leg name="leg5" x="0.09" y="0.065" angle="0.7854" side="-1" />    <!-- Front Right -->
+  <xacro:leg name="0" x="-0.09" y="-0.065" angle="-2.35619" side="1" /> <!-- Back Left -->
+  <xacro:leg name="1" x="0.0" y="-0.09" angle="-1.5708" side="1" />     <!-- Left -->
+  <xacro:leg name="2" x="0.09" y="-0.065" angle="-0.7854" side="1" />   <!-- Front Left -->
+  <xacro:leg name="3" x="-0.09" y="0.065" angle="2.35619" side="-1" />  <!-- Back Right -->
+  <xacro:leg name="4" x="0.0" y="0.09" angle="1.5708" side="-1" />      <!-- Right -->
+  <xacro:leg name="5" x="0.09" y="0.065" angle="0.7854" side="-1" />    <!-- Front Right -->
 </robot>
